File: pcb/sma_measurement.kicad_sch (KiCad schematic)
At the start: 2 parts, among them U8 MCP3008

Commit message: final version schematic?
Connections:
- net FG One Voltage Sensing/FG_One_G34: now reaches U8.5 (CH4)
- net FG One Voltage Sensing/FG_One_G8: now reaches U8.6 (CH5)
- net FG One Voltage Sensing/FG_One_SP: now reaches U8.7 (CH6)
- net FG One Voltage Sensing/FG_One_WS: now reaches U8.8 (CH7)
Other:
- sheet FG Flex Voltage Sensing ports: added I_FG_Flex; removed I_FG_FLEX
- sheet FG One Voltage Sensing ports: added FG_One_G34, FG_One_G8, FG_One_SP, FG_One_WS; removed none
- company: (none) -> /dev/tal e.V.
- title: (none) -> SMA Voltage Measurement ADC
- moved on the sheet: C19
Changed lines of the file:
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@@
 (kicad_sch (version 20230121) (generator eeschema)
   (paper "A4")
+  (title_block
+    (title "SMA Voltage Measurement ADC")
+    (date "2023-12-09")
+    (rev "0.5")
+    (company "/dev/tal e.V.")
+  )
+  (wire (pts (xy 152.4 99.06) (xy 154.94 99.06))
+    (stroke (width 0) (type default))
+  )
   (wire (pts (xy 185.42 99.06) (xy 185.42 104.14))
     (stroke (width 0) (type default))
   )
+  (wire (pts (xy 160.02 91.44) (xy 165.1 91.44))
+    (stroke (width 0) (type default))
+  )
   (wire (pts (xy 116.84 63.5) (xy 127 63.5))
     (stroke (width 0) (type default))
@@
     (stroke (width 0) (type default))
   )
+  (wire (pts (xy 152.4 114.3) (xy 162.56 114.3))
+    (stroke (width 0) (type default))
+  )
   (wire (pts (xy 177.8 99.06) (xy 177.8 104.14))
     (stroke (width 0) (type default))
   )
+  (wire (pts (xy 116.84 106.68) (xy 127 106.68))
+    (stroke (width 0) (type default))
+  )
   (wire (pts (xy 160.02 78.74) (xy 165.1 78.74))
     (stroke (width 0) (type default))
@@
     (stroke (width 0) (type default))
   )
+  (wire (pts (xy 152.4 104.14) (xy 157.48 104.14))
+    (stroke (width 0) (type default))
+  )
+  (wire (pts (xy 154.94 99.06) (xy 154.94 86.36))
+    (stroke (width 0) (type default))
+  )
+  (wire (pts (xy 154.94 86.36) (xy 165.1 86.36))
+    (stroke (width 0) (type default))
+  )
   (wire (pts (xy 195.58 83.82) (xy 203.2 83.82))
     (stroke (width 0) (type default))
@@
     (stroke (width 0) (type default))
   )
+  (wire (pts (xy 157.48 104.14) (xy 157.48 88.9))
+    (stroke (width 0) (type default))
+  )
   (wire (pts (xy 152.4 60.96) (xy 160.02 60.96))
     (stroke (width 0) (type default))
   )
+  (wire (pts (xy 160.02 109.22) (xy 160.02 91.44))
+    (stroke (width 0) (type default))
+  )
   (wire (pts (xy 162.56 76.2) (xy 162.56 55.88))
     (stroke (width 0) (type default))
@@
     (stroke (width 0) (type default))
   )
-  (wire (pts (xy 242.062 39.624) (xy 242.062 44.704))
-    (stroke (width 0) (type default))
-  )
-  (wire (pts (xy 242.062 29.464) (xy 242.062 34.544))
+  (wire (pts (xy 241.3 40.64) (xy 241.3 45.72))
+    (stroke (width 0) (type default))
+  )
+  (wire (pts (xy 241.3 30.48) (xy 241.3 35.56))
     (stroke (width 0) (type default))
   )
@@
     (stroke (width 0) (type default))
   )
+  (wire (pts (xy 152.4 109.22) (xy 160.02 109.22))
+    (stroke (width 0) (type default))
+  )
+  (wire (pts (xy 157.48 88.9) (xy 165.1 88.9))
+    (stroke (width 0) (type default))
+  )
   (wire (pts (xy 154.94 83.82) (xy 165.1 83.82))
+    (stroke (width 0) (type default))
+  )
+  (wire (pts (xy 162.56 93.98) (xy 165.1 93.98))
+    (stroke (width 0) (type default))
+  )
+  (wire (pts (xy 162.56 114.3) (xy 162.56 93.98))
     (stroke (width 0) (type default))
   )
@@
     )
   )
-  (symbol (lib_id "power:+5V") (at 242.062 29.464 0) (unit 1)
+  (symbol (lib_id "power:+5V") (at 241.3 30.48 0) (unit 1)
     (in_bom yes) (on_board yes) (dnp no)
-    (property "Reference" "#PWR061" (at 242.062 33.274 0)
-      (effects (font (size 1.27 1.27)) hide)
-    )
-    (property "Value" "+5V" (at 242.062 26.162 0)
+    (property "Reference" "#PWR061" (at 241.3 34.29 0)
+      (effects (font (size 1.27 1.27)) hide)
+    )
+    (property "Value" "+5V" (at 241.3 27.178 0)
       (effects (font (size 1.27 1.27)))
     )
-    (property "Footprint" "" (at 242.062 29.464 0)
-      (effects (font (size 1.27 1.27)) hide)
-    )
-    (property "Datasheet" "" (at 242.062 29.464 0)
+    (property "Footprint" "" (at 241.3 30.48 0)
+      (effects (font (size 1.27 1.27)) hide)
+    )
+    (property "Datasheet" "" (at 241.3 30.48 0)
       (effects (font (size 1.27 1.27)) hide)
     )
@@
     )
   )
-  (symbol (lib_id "Device:C_Small") (at 242.062 37.084 0) (unit 1)
+  (symbol (lib_id "Device:C_Small") (at 241.3 38.1 0) (unit 1)
     (in_bom yes) (on_board yes) (dnp no)
-    (property "Reference" "C19" (at 242.316 35.56 0)
-      (effects (font (size 1.27 1.27)) (justify left))
-    )
-    (property "Value" "1uF" (at 242.316 38.608 0)
-      (effects (font (size 1.27 1.27)) (justify left))
-    )
-    (property "Footprint" "Capacitor_THT:C_Disc_D4.7mm_W2.5mm_P5.00mm" (at 242.062 37.084 0)
-      (effects (font (size 1.27 1.27)) hide)
-    )
-    (property "Datasheet" "https://product.tdk.com/en/system/files?file=dam/doc/product/capacitor/ceramic/lead-mlcc/catalog/leadmlcc_halogenfree_fg_en.pdf" (at 242.062 37.084 0)
-      (effects (font (size 1.27 1.27)) hide)
-    )
-    (property "Manufacturer" "TDK Corporation" (at 242.062 37.084 0)
-      (effects (font (size 1.27 1.27)) hide)
-    )
-    (property "Part Nr." "FG28X5R1H105KRT06" (at 242.062 37.084 0)
+    (property "Reference" "C19" (at 241.554 36.576 0)
+      (effects (font (size 1.27 1.27)) (justify left))
+    )
+    (property "Value" "1uF" (at 241.554 39.624 0)
+      (effects (font (size 1.27 1.27)) (justify left))
+    )
+    (property "Footprint" "Capacitor_THT:C_Disc_D4.7mm_W2.5mm_P5.00mm" (at 241.3 38.1 0)
+      (effects (font (size 1.27 1.27)) hide)
+    )
+    (property "Datasheet" "https://product.tdk.com/en/system/files?file=dam/doc/product/capacitor/ceramic/lead-mlcc/catalog/leadmlcc_halogenfree_fg_en.pdf" (at 241.3 38.1 0)
+      (effects (font (size 1.27 1.27)) hide)
+    )
+    (property "Manufacturer" "TDK Corporation" (at 241.3 38.1 0)
+      (effects (font (size 1.27 1.27)) hide)
+    )
+    (property "Part Nr." "FG28X5R1H105KRT06" (at 241.3 38.1 0)
       (effects (font (size 1.27 1.27)) hide)
     )
@@
     )
   )
-  (symbol (lib_id "power:GND") (at 242.062 44.704 0) (unit 1)
+  (symbol (lib_id "power:GND") (at 241.3 45.72 0) (unit 1)
     (in_bom yes) (on_board yes) (dnp no) (fields_autoplaced)
-    (property "Reference" "#PWR062" (at 242.062 51.054 0)
-      (effects (font (size 1.27 1.27)) hide)
-    )
-    (property "Value" "GND" (at 242.062 49.53 0)
-      (effects (font (size 1.27 1.27)) hide)
-    )
-    (property "Footprint" "" (at 242.062 44.704 0)
-      (effects (font (size 1.27 1.27)) hide)
-    )
-    (property "Datasheet" "" (at 242.062 44.704 0)
+    (property "Reference" "#PWR062" (at 241.3 52.07 0)
+      (effects (font (size 1.27 1.27)) hide)
+    )
+    (property "Value" "GND" (at 241.3 50.546 0)
+      (effects (font (size 1.27 1.27)) hide)
+    )
+    (property "Footprint" "" (at 241.3 45.72 0)
+      (effects (font (size 1.27 1.27)) hide)
+    )
+    (property "Datasheet" "" (at 241.3 45.72 0)
       (effects (font (size 1.27 1.27)) hide)
     )
@@
       (effects (font (size 1.27 1.27)) (justify left))
     )
+    (pin "FG_One_WS" output (at 152.4 114.3 0)
+      (effects (font (size 1.27 1.27)) (justify right))
+    )
+    (pin "FG_One_SP" output (at 152.4 109.22 0)
+      (effects (font (size 1.27 1.27)) (justify right))
+    )
+    (pin "FG_One_G8" output (at 152.4 104.14 0)
+      (effects (font (size 1.27 1.27)) (justify right))
+    )
+    (pin "FG_One_G34" output (at 152.4 99.06 0)
+      (effects (font (size 1.27 1.27)) (justify right))
+    )
     (instances
       (project "fg_lampe"
@@
       (effects (font (size 1.27 1.27)) (justify right))
     )
-    (pin "I_FG_FLEX" input (at 127 63.5 180)
-      (effects (font (size 1.27 1.27)) (justify left))
-    )
+    (pin "I_FG_Flex" input (at 127 63.5 180)
+      (effects (font (size 1.27 1.27)) (justify left))
+    )
