File: pcb/fg-one_current_source.kicad_sch (KiCad schematic)
At the start: 26 parts, among them Q3 BC547, Q4 IRF9540N, Q5 IRF9540N, U6 LM358, U9 TL071

Commit message: finals in schematic
Parts:
- added J13: Shunt Pin FG One, Connector_PinHeader_2.54mm:PinHeader_1x02_P2.54mm_Vertical, symbol Connector:Conn_01x02_Pin
- C13, C14: footprint Capacitor_THT:C_Disc_D5.1mm_W3.2mm_P5.00mm -> Capacitor_THT:C_Disc_D5.0mm_W2.5mm_P2.50mm
Connections:
- net at Q4.2 (D), R18.1, R19.1: now also J13.2 (Pin_2)
- net at Q5.3 (S), R16.2, R18.2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: now also J13.1 (Pin_1)
Changed lines of the file:
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@@
   (junction (at 149.86 119.38) (diameter 0) (color 0 0 0 0)
   )
+  (junction (at 157.48 111.76) (diameter 0) (color 0 0 0 0)
+  )
   (junction (at 205.74 104.14) (diameter 0) (color 0 0 0 0)
   )
@@
   )
   (junction (at 228.6 104.14) (diameter 0) (color 0 0 0 0)
+  )
+  (junction (at 157.48 96.52) (diameter 0) (color 0 0 0 0)
   )
   (junction (at 121.92 78.74) (diameter 0) (color 0 0 0 0)
@@
     (stroke (width 0) (type default))
   )
-  (wire (pts (xy 149.86 111.76) (xy 162.56 111.76))
+  (wire (pts (xy 149.86 111.76) (xy 157.48 111.76))
     (stroke (width 0) (type default))
   )
@@
     (stroke (width 0) (type default))
   )
+  (wire (pts (xy 157.48 102.616) (xy 157.48 96.52))
+    (stroke (width 0) (type default))
+  )
   (wire (pts (xy 20.32 45.72) (xy 20.32 50.8))
     (stroke (width 0) (type default))
@@
     (stroke (width 0) (type default))
   )
+  (wire (pts (xy 157.48 105.156) (xy 157.48 111.76))
+    (stroke (width 0) (type default))
+  )
   (wire (pts (xy 121.92 119.38) (xy 121.92 124.46))
     (stroke (width 0) (type default))
@@
     (stroke (width 0) (type default))
   )
+  (wire (pts (xy 160.02 105.156) (xy 157.48 105.156))
+    (stroke (width 0) (type default))
+  )
   (wire (pts (xy 121.92 63.5) (xy 121.92 71.12))
     (stroke (width 0) (type default))
@@
     (stroke (width 0) (type default))
   )
+  (wire (pts (xy 157.48 111.76) (xy 162.56 111.76))
+    (stroke (width 0) (type default))
+  )
   (wire (pts (xy 203.2 50.8) (xy 203.2 60.96))
     (stroke (width 0) (type default))
@@
     (stroke (width 0) (type default))
   )
-  (wire (pts (xy 149.86 96.52) (xy 162.56 96.52))
+  (wire (pts (xy 149.86 96.52) (xy 157.48 96.52))
     (stroke (width 0) (type default))
   )
@@
     (stroke (width 0) (type default))
   )
+  (wire (pts (xy 157.48 96.52) (xy 162.56 96.52))
+    (stroke (width 0) (type default))
+  )
   (wire (pts (xy 228.6 104.14) (xy 261.62 104.14))
+    (stroke (width 0) (type default))
+  )
+  (wire (pts (xy 160.02 102.616) (xy 157.48 102.616))
     (stroke (width 0) (type default))
   )
@@
       (effects (font (size 1.27 1.27)) (justify left))
     )
-    (property "Footprint" "Capacitor_THT:C_Disc_D5.1mm_W3.2mm_P5.00mm" (at 38.1 38.1 0)
+    (property "Footprint" "Capacitor_THT:C_Disc_D5.0mm_W2.5mm_P2.50mm" (at 38.1 38.1 0)
       (effects (font (size 1.27 1.27)) hide)
     )
@@
       (effects (font (size 1.27 1.27)) (justify left))
     )
-    (property "Footprint" "Capacitor_THT:C_Disc_D5.1mm_W3.2mm_P5.00mm" (at 203.2 63.5 0)
+    (property "Footprint" "Capacitor_THT:C_Disc_D5.0mm_W2.5mm_P2.50mm" (at 203.2 63.5 0)
       (effects (font (size 1.27 1.27)) hide)
     )
@@
     )
   )
+  (symbol (lib_id "Connector:Conn_01x02_Pin") (at 165.1 105.156 180) (unit 1)
+    (in_bom yes) (on_board yes) (dnp no)
+    (property "Reference" "J13" (at 166.37 102.616 0)
+      (effects (font (size 1.27 1.27)) (justify right))
+    )
+    (property "Value" "Shunt Pin FG One" (at 160.02 107.696 0)
+      (effects (font (size 1.27 1.27)) (justify right))
+    )
+    (property "Footprint" "Connector_PinHeader_2.54mm:PinHeader_1x02_P2.54mm_Vertical" (at 165.1 105.156 0)
+      (effects (font (size 1.27 1.27)) hide)
+    )
+    (property "Datasheet" "~" (at 165.1 105.156 0)
+      (effects (font (size 1.27 1.27)) hide)
+    )
+    (pin "2")
+    (pin "1")
+    (instances
+      (project "fg_lampe"
+        (path "/6ce7d73a-8297-412b-a1cf-6113d41486fd/ba76f9dc-1045-4df8-971c-12fc9c8a3a7f"
+          (reference "J13") (unit 1)
+        )
+      )
+    )
+  )
   (symbol (lib_id "Device:R_Small") (at 149.86 104.14 0) (unit 1)
     (in_bom yes) (on_board yes) (dnp no) (fields_autoplaced)
@@
       (effects (font (size 1.27 1.27)) (justify left))
     )
-    (property "Footprint" "Capacitor_THT:C_Disc_D5.1mm_W3.2mm_P5.00mm" (at 195.58 63.5 0)
+    (property "Footprint" "Capacitor_THT:C_Disc_D5.0mm_W2.5mm_P2.50mm" (at 195.58 63.5 0)
       (effects (font (size 1.27 1.27)) hide)
     )
@@
       (effects (font (size 1.27 1.27)) (justify left))
     )
-    (property "Footprint" "Capacitor_THT:C_Disc_D5.1mm_W3.2mm_P5.00mm" (at 30.48 38.1 0)
-      (effects (font (size 1.27 1.27)) hide)
-    )
+    (property "Footprint" "Capacitor_THT:C_Disc_D5.0mm_W2.5mm_P2.50mm" (at 30.48 38.1 0)
+      (effects (font (size 1.27 1.27)) hide)
+    )
