File: pcb/fg_lampe.kicad_sch (KiCad schematic)
At the start: 63 parts, among them J1 ISP Port, J11 SPI Debug Pins, J2 1792863, J3 1792863, J4 1792863, J5 1792876, J6 PWR Control, J7 RX/TX, J8 I^{2}C Debug, Q1 IRLZ540N, Q2 IRLZ540N, SW1 Reset Button, U1 ATmega328P-P, U2 L7805, U3 MAX1044, U4 MAX1044, U5 MIC4427, U6 MCP4812, U7 MCP3008, Y1 16MHz

Commit message: finals in schematic
Parts:
- added J12: DAC Tespins, Connector_PinHeader_2.54mm:PinHeader_1x03_P2.54mm_Vertical, symbol Connector:Conn_01x03_Pin
- C1, C2, C3: value 100nF -> 0.1uF; footprint Capacitor_THT:C_Disc_D3.8mm_W2.6mm_P2.50mm -> Capacitor_THT:C_Disc_D5.0mm_W2.5mm_P2.50mm
- C10, C13, C17, C4, C6, C8, C9: footprint Capacitor_THT:C_Disc_D5.1mm_W3.2mm_P5.00mm -> Capacitor_THT:C_Disc_D5.0mm_W2.5mm_P2.50mm
- C18: footprint Capacitor_THT:CP_Radial_Tantal_D6.0mm_P2.50mm -> Capacitor_THT:CP_Radial_Tantal_D5.0mm_P5.00mm
- C19, C7: footprint Capacitor_THT:C_Disc_D4.7mm_W2.5mm_P5.00mm -> Capacitor_THT:C_Disc_D3.8mm_W2.6mm_P2.50mm
- Y1: Part Nr.  ATS16A -> AS-16.000-18
Connections:
- net GND: now also J12.2 (Pin_2)
- net V_{A}: now also J12.3 (Pin_3)
- net V_{B}: now also J12.1 (Pin_1)
Changed lines of the file:
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@@
     (stroke (width 0) (type default))
   )
+  (wire (pts (xy 190.5 127) (xy 180.34 127))
+    (stroke (width 0) (type default))
+  )
   (wire (pts (xy 93.98 110.49) (xy 96.52 110.49))
     (stroke (width 0) (type default))
@@
     (stroke (width 0) (type default))
   )
+  (wire (pts (xy 182.88 129.54) (xy 190.5 129.54))
+    (stroke (width 0) (type default))
+  )
   (wire (pts (xy 274.32 99.06) (xy 281.94 99.06))
     (stroke (width 0) (type default))
@@
     (stroke (width 0) (type default))
   )
+  (wire (pts (xy 180.34 127) (xy 180.34 132.08))
+    (stroke (width 0) (type default))
+  )
   (wire (pts (xy 243.84 55.88) (xy 251.46 55.88))
     (stroke (width 0) (type default))
@@
     (stroke (width 0) (type default))
   )
+  (wire (pts (xy 182.88 124.46) (xy 190.5 124.46))
+    (stroke (width 0) (type default))
+  )
   (wire (pts (xy 120.65 92.71) (xy 120.65 95.25))
     (stroke (width 0) (type default))
@@
     (effects (font (size 0.5 0.5)) (justify left bottom))
   )
+  (label "V_{A}" (at 182.88 124.46 0) (fields_autoplaced)
+    (effects (font (size 1.27 1.27)) (justify left bottom))
+  )
   (label "SCL" (at 71.12 68.58 180) (fields_autoplaced)
     (effects (font (size 1.27 1.27)) (justify right bottom))
@@
     (effects (font (size 1.27 1.27)) (justify right bottom))
   )
+  (label "V_{B}" (at 182.88 129.54 0) (fields_autoplaced)
+    (effects (font (size 1.27 1.27)) (justify left bottom))
+  )
   (label "warm_led_to_gnd" (at 210.82 76.2 180) (fields_autoplaced)
     (effects (font (size 1.27 1.27)) (justify right bottom))
@@
       (effects (font (size 1.27 1.27)) (justify left))
     )
-    (property "Footprint" "Capacitor_THT:C_Disc_D5.1mm_W3.2mm_P5.00mm" (at 38.1 132.08 0)
+    (property "Footprint" "Capacitor_THT:C_Disc_D5.0mm_W2.5mm_P2.50mm" (at 38.1 132.08 0)
       (effects (font (size 1.27 1.27)) hide)
     )
@@
       (effects (font (size 1.27 1.27)) (justify left))
     )
-    (property "Footprint" "Capacitor_THT:C_Disc_D5.1mm_W3.2mm_P5.00mm" (at 86.36 27.94 0)
+    (property "Footprint" "Capacitor_THT:C_Disc_D5.0mm_W2.5mm_P2.50mm" (at 86.36 27.94 0)
       (effects (font (size 1.27 1.27)) hide)
     )
@@
       (effects (font (size 1.27 1.27)) (justify left))
     )
-    (property "Footprint" "Capacitor_THT:C_Disc_D4.7mm_W2.5mm_P5.00mm" (at 76.2 27.94 0)
+    (property "Footprint" "Capacitor_THT:C_Disc_D3.8mm_W2.6mm_P2.50mm" (at 76.2 27.94 0)
       (effects (font (size 1.27 1.27)) hide)
     )
@@
       (effects (font (size 1.27 1.27)) (justify left))
     )
-    (property "Value" "100nF" (at 20.32 39.878 0)
+    (property "Value" "0.1uF" (at 20.32 39.878 0)
       (effects (font (size 1.27 1.27)) (justify left))
     )
-    (property "Footprint" "Capacitor_THT:C_Disc_D3.8mm_W2.6mm_P2.50mm" (at 20.32 38.1 0)
+    (property "Footprint" "Capacitor_THT:C_Disc_D5.0mm_W2.5mm_P2.50mm" (at 20.32 38.1 0)
       (effects (font (size 1.27 1.27)) hide)
     )
@@
       (effects (font (size 1.27 1.27)) (justify left))
     )
-    (property "Footprint" "Capacitor_THT:C_Disc_D5.1mm_W3.2mm_P5.00mm" (at 78.74 175.26 0)
+    (property "Footprint" "Capacitor_THT:C_Disc_D5.0mm_W2.5mm_P2.50mm" (at 78.74 175.26 0)
       (effects (font (size 1.27 1.27)) hide)
     )
@@
   (symbol (lib_id "Device:C_Small") (at 91.44 118.11 90) (unit 1)
     (in_bom yes) (on_board yes) (dnp no)
-    (property "Reference" "C12" (at 93.218 117.348 90)
+    (property "Reference" "C12" (at 93.98 117.348 90)
       (effects (font (size 1.27 1.27)))
     )
@@
   (symbol (lib_id "Device:C_Small") (at 91.44 110.49 90) (unit 1)
     (in_bom yes) (on_board yes) (dnp no)
-    (property "Reference" "C11" (at 93.218 109.728 90)
+    (property "Reference" "C11" (at 93.98 109.728 90)
       (effects (font (size 1.27 1.27)))
     )
@@
       (effects (font (size 1.27 1.27)) (justify left))
     )
-    (property "Value" "100nF" (at 22.86 100.838 0)
+    (property "Value" "0.1uF" (at 22.86 100.838 0)
       (effects (font (size 1.27 1.27)) (justify left))
     )
-    (property "Footprint" "Capacitor_THT:C_Disc_D3.8mm_W2.6mm_P2.50mm" (at 22.86 99.06 0)
+    (property "Footprint" "Capacitor_THT:C_Disc_D5.0mm_W2.5mm_P2.50mm" (at 22.86 99.06 0)
       (effects (font (size 1.27 1.27)) hide)
     )
@@
       (effects (font (size 1.27 1.27)) (justify left))
     )
-    (property "Footprint" "Capacitor_THT:C_Disc_D5.1mm_W3.2mm_P5.00mm" (at 63.5 132.08 0)
+    (property "Footprint" "Capacitor_THT:C_Disc_D5.0mm_W2.5mm_P2.50mm" (at 63.5 132.08 0)
       (effects (font (size 1.27 1.27)) hide)
     )
@@
     )
   )
+  (symbol (lib_id "power:GND") (at 180.34 132.08 0) (unit 1)
+    (in_bom yes) (on_board yes) (dnp no) (fields_autoplaced)
+    (property "Reference" "#PWR0177" (at 180.34 138.43 0)
+      (effects (font (size 1.27 1.27)) hide)
+    )
+    (property "Value" "GND" (at 180.34 136.906 0)
+      (effects (font (size 1.27 1.27)) hide)
+    )
+    (property "Footprint" "" (at 180.34 132.08 0)
+      (effects (font (size 1.27 1.27)) hide)
+    )
+    (property "Datasheet" "" (at 180.34 132.08 0)
+      (effects (font (size 1.27 1.27)) hide)
+    )
+    (pin "1")
+    (instances
+      (project "fg_lampe"
+        (path "/6ce7d73a-8297-412b-a1cf-6113d41486fd"
+          (reference "#PWR0177") (unit 1)
+        )
+      )
+    )
+  )
   (symbol (lib_id "Device:C_Polarized_Small") (at 142.24 137.16 0) (unit 1)
     (in_bom yes) (on_board yes) (dnp no) (fields_autoplaced)
@@
       (effects (font (size 1.27 1.27)) (justify left))
     )
-    (property "Footprint" "Capacitor_THT:CP_Radial_Tantal_D6.0mm_P2.50mm" (at 142.24 137.16 0)
+    (property "Footprint" "Capacitor_THT:CP_Radial_Tantal_D5.0mm_P5.00mm" (at 142.24 137.16 0)
       (effects (font (size 1.27 1.27)) hide)
     )
@@
     )
   )
+  (symbol (lib_id "Connector:Conn_01x03_Pin") (at 195.58 127 180) (unit 1)
+    (in_bom yes) (on_board yes) (dnp no)
+    (property "Reference" "J12" (at 193.802 123.444 0)
+      (effects (font (size 1.27 1.27)) (justify right))
+    )
+    (property "Value" "DAC Tespins" (at 185.42 132.08 0)
+      (effects (font (size 1.27 1.27)) (justify right))
+    )
+    (property "Footprint" "Connector_PinHeader_2.54mm:PinHeader_1x03_P2.54mm_Vertical" (at 195.58 127 0)
+      (effects (font (size 1.27 1.27)) hide)
+    )
+    (property "Datasheet" "~" (at 195.58 127 0)
+      (effects (font (size 1.27 1.27)) hide)
+    )
+    (pin "1")
+    (pin "2")
+    (pin "3")
+    (instances
+      (project "fg_lampe"
+        (path "/6ce7d73a-8297-412b-a1cf-6113d41486fd"
+          (reference "J12") (unit 1)
+        )
+      )
+    )
+  )
   (symbol (lib_id "power:+5V") (at 43.18 20.32 0) (unit 1)
     (in_bom yes) (on_board yes) (dnp no)
@@
       (effects (font (size 1.27 1.27)) (justify left))
     )
-    (property "Footprint" "Capacitor_THT:C_Disc_D4.7mm_W2.5mm_P5.00mm" (at 223.52 86.36 0)
+    (property "Footprint" "Capacitor_THT:C_Disc_D3.8mm_W2.6mm_P2.50mm" (at 223.52 86.36 0)
       (effects (font (size 1.27 1.27)) hide)
     )
@@
       (effects (font (size 1.27 1.27)) (justify left))
     )
-    (property "Footprint" "Capacitor_THT:C_Disc_D5.1mm_W3.2mm_P5.00mm" (at 134.62 137.16 0)
+    (property "Footprint" "Capacitor_THT:C_Disc_D5.0mm_W2.5mm_P2.50mm" (at 134.62 137.16 0)
       (effects (font (size 1.27 1.27)) hide)
     )
@@
       (effects (font (size 1.27 1.27)) (justify left))
     )
-    (property "Footprint" "Capacitor_THT:C_Disc_D5.1mm_W3.2mm_P5.00mm" (at 96.52 27.94 0)
+    (property "Footprint" "Capacitor_THT:C_Disc_D5.0mm_W2.5mm_P2.50mm" (at 96.52 27.94 0)
       (effects (font (size 1.27 1.27)) hide)
     )
@@
       (effects (font (size 1.27 1.27)) (justify left))
     )
-    (property "Footprint" "Capacitor_THT:C_Disc_D5.1mm_W3.2mm_P5.00mm" (at 78.74 139.7 0)
+    (property "Footprint" "Capacitor_THT:C_Disc_D5.0mm_W2.5mm_P2.50mm" (at 78.74 139.7 0)
       (effects (font (size 1.27 1.27)) hide)
     )
@@
       (effects (font (size 1.27 1.27)) (justify left))
     )
-    (property "Value" "100nF" (at 15.24 100.838 0)
+    (property "Value" "0.1uF" (at 15.24 100.838 0)
       (effects (font (size 1.27 1.27)) (justify left))
     )
-    (property "Footprint" "Capacitor_THT:C_Disc_D3.8mm_W2.6mm_P2.50mm" (at 15.24 99.06 0)
+    (property "Footprint" "Capacitor_THT:C_Disc_D5.0mm_W2.5mm_P2.50mm" (at 15.24 99.06 0)
       (effects (font (size 1.27 1.27)) hide)
     )
@@
       (effects (font (size 1.27 1.27)) hide)
     )
-    (property "Datasheet" "https://www.ctscorp.com/wp-content/uploads/ATS-ATSSM.pdf" (at 83.82 114.3 0)
+    (property "Datasheet" "https://www.raltron.com/webproducts/specs/CRYSTAL/AS-16.000-18.pdf" (at 83.82 114.3 0)
       (effects (font (size 1.27 1.27)) hide)
     )
-    (property "Part Nr. " "ATS16A" (at 83.82 114.3 90)
+    (property "Part Nr. " "AS-16.000-18" (at 83.82 114.3 90)
       (effects (font (size 1.27 1.27)) hide)
     )
