File: pcb/fg_lampe.kicad_sch (KiCad schematic)
At the start: 64 parts, among them J1 ISP Port, J11 SPI Debug Pins, J12 DAC Tespins, J2 1792863, J3 1792863, J4 1792863, J5 1792876, J6 PWR Control, J7 RX/TX, J8 I^{2}C Debug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

Commit message: start pcb
Parts:
- added HS1: Heatsink_Pad, Heatsink:Heatsink_Stonecold_HS-132_32x14mm_2xFixation1.5mm, symbol Mechanical:Heatsink_Pad
- U2: footprint Package_TO_SOT_THT:TO-220-3_Horizontal_TabDown -> Package_TO_SOT_THT:TO-220-3_Vertical
Connections:
- no-connect marks 5 -> 6
Changed lines of the file:
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@@
   (junction (at 45.72 157.48) (diameter 0) (color 0 0 0 0)
   )
+  (no_connect (at 17.78 129.54))
   (no_connect (at 83.82 182.88))
   (no_connect (at 83.82 142.24))
@@
     )
   )
+  (symbol (lib_id "Mechanical:Heatsink_Pad") (at 17.78 127 0) (unit 1)
+    (in_bom yes) (on_board yes) (dnp no) (fields_autoplaced)
+    (property "Reference" "HS1" (at 21.59 125.095 0)
+      (effects (font (size 1.27 1.27)) (justify left))
+    )
+    (property "Value" "Heatsink_Pad" (at 21.59 127.635 0)
+      (effects (font (size 1.27 1.27)) (justify left))
+    )
+    (property "Footprint" "Heatsink:Heatsink_Stonecold_HS-132_32x14mm_2xFixation1.5mm" (at 18.0848 128.27 0)
+      (effects (font (size 1.27 1.27)) hide)
+    )
+    (property "Datasheet" "~" (at 18.0848 128.27 0)
+      (effects (font (size 1.27 1.27)) hide)
+    )
+    (pin "1")
+    (instances
+      (project "fg_lampe"
+        (path "/6ce7d73a-8297-412b-a1cf-6113d41486fd"
+          (reference "HS1") (unit 1)
+        )
+      )
+    )
+  )
   (symbol (lib_id "Device:R_Small") (at 172.72 86.36 90) (unit 1)
     (in_bom yes) (on_board yes) (dnp no)
@@
       (effects (font (size 1.27 1.27)))
     )
-    (property "Footprint" "Package_TO_SOT_THT:TO-220-3_Horizontal_TabDown" (at 51.435 128.27 0)
+    (property "Footprint" "Package_TO_SOT_THT:TO-220-3_Vertical" (at 51.435 128.27 0)
       (effects (font (size 1.27 1.27) italic) (justify left) hide)
     )
