File: pcb/fg_one_voltage_sensing.kicad_sch (KiCad schematic)
At the start: 25 parts

Commit message: final version schematic?
Other:
- company: (none) -> /dev/tal e.V.
- title: (none) -> FG One Amplifier Circuit
Changed lines of the file:
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@@
 (kicad_sch (version 20230121) (generator eeschema)
   (paper "A4")
+  (title_block
+    (title "FG One Amplifier Circuit")
+    (date "2023-12-09")
+    (rev "0.5")
+    (company "/dev/tal e.V.")
+  )
   (junction (at 76.2 86.36) (diameter 0) (color 0 0 0 0)
   )

Commit message: finals in schematic
Parts:
- C13, C14: footprint Capacitor_THT:C_Disc_D5.1mm_W3.2mm_P5.00mm -> Capacitor_THT:C_Disc_D5.0mm_W2.5mm_P2.50mm
Changed lines of the file:
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@@
       (effects (font (size 1.27 1.27)) (justify left))
     )
-    (property "Footprint" "Capacitor_THT:C_Disc_D5.1mm_W3.2mm_P5.00mm" (at 246.38 38.1 0)
+    (property "Footprint" "Capacitor_THT:C_Disc_D5.0mm_W2.5mm_P2.50mm" (at 246.38 38.1 0)
       (effects (font (size 1.27 1.27)) hide)
     )
@@
       (effects (font (size 1.27 1.27)) (justify left))
     )
-    (property "Footprint" "Capacitor_THT:C_Disc_D5.1mm_W3.2mm_P5.00mm" (at 254 38.1 0)
-      (effects (font (size 1.27 1.27)) hide)
-    )
+    (property "Footprint" "Capacitor_THT:C_Disc_D5.0mm_W2.5mm_P2.50mm" (at 254 38.1 0)
+      (effects (font (size 1.27 1.27)) hide)
+    )
